File: kicad/_autosave-matesepia.kicad_pcb (KiCad board)
At the start: 2 copper layers, 227.4 x 131.5 mm, 63 parts

Commit message: Solving for push
Parts:
- moved D25 6.66 mm to (184.8, 99.2)
- moved D4 6.66 mm to (82.0, 55.7)
- moved D5 6.66 mm to (90.8, 38.8)
- moved D6 6.66 mm to (92.2, 78.3)
- moved D7 6.66 mm to (102.4, 62.3)
- moved D9 6.66 mm to (103.6, 95.8)
- moved MCU1 6.66 mm to (154.4, 101.8)
- moved S10 6.66 mm to (116.5, 75.5)
- moved S25 6.66 mm to (182.1, 95.0)
- moved S6 6.66 mm to (94.9, 74.1)
- moved S9 6.66 mm to (106.3, 91.5)
- moved D11 6.66 mm to (124.0, 63.7)
- moved D12 6.66 mm to (123.9, 99.2)
- moved D13 6.66 mm to (134.2, 83.2)
- moved D15 6.66 mm to (251.7, 60.7)
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Routing:
- removed copper zone on F.Cu, net (none)
