File: kicad/metasepia_good.kicad_pcb (KiCad board)
At the start: 2 copper layers, 227.4 x 131.5 mm, 63 parts

Commit message: properly remaking traces from scratch. Half done.
Parts:
- moved D29 35.7 mm to (177.5, 160.4)
- moved D18 35.7 mm to (188.5, 66.3)
- moved S22 35.7 mm to (173.0, 119.0)
- moved S26 35.7 mm to (142.5, 106.5)
- moved S9 35.7 mm to (76.9, 119.0)
- moved D7 35.7 mm to (73.0, 89.8)
- moved S2 35.7 mm to (29.6, 83.5)
- moved D14 35.7 mm to (229.5, 105.7)
- moved S12 35.7 mm to (97.2, 122.5)
- moved S29 35.7 mm to (174.9, 156.2)
- moved D10 35.7 mm to (84.4, 107.2)
- moved D2 35.7 mm to (27.7, 88.2)
- moved S27 35.7 mm to (75.1, 156.2)
- moved S3 35.7 mm to (46.2, 95.6)
- moved D13 35.7 mm to (104.7, 110.7)
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Routing:
- net P7: track 0.00 -> 218.1 mm, vias 0 -> 2
- net P6: track 0.00 -> 202.6 mm, vias 0 -> 3
- net P2: track 0.00 -> 152.1 mm, vias 0 -> 3
- net P5: track 0.00 -> 151.9 mm, vias 0 -> 2
- net P4: track 0.00 -> 145.6 mm, vias 0 -> 3
- net P8: track 0.00 -> 135.3 mm, vias 0 -> 1
- net P0: track 0.00 -> 133.6 mm, vias 0 -> 2
- net P3: track 0.00 -> 100.0 mm, vias 0 -> 2
- net P1: track 0.00 -> 99.8 mm, vias 0 -> 2
- net P9: track 0.00 -> 61.3 mm
- net P10: track 0.00 -> 41.5 mm
- net pinky_home: track 0.00 -> 10.3 mm
- net pinky_bottom: track 0.00 -> 10.3 mm
- net mirror_pinky_bottom: track 0.00 -> 10.2 mm
- net mirror_pinky_home: track 0.00 -> 10.2 mm
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
Commit message: almost finish routing
Parts:
- MCU1: footprint frequent:xiao-ble-smd-cutout -> frequent:xiao-smd
- S1, S10, S11, S12, S13, S14, S15, S16, S17, S18, S19, S2, S20, S21, S22, S23, S24, S25, S26, S27, S28, S29, S3, S30, S4, S5, S6, S7, S8, S9: footprint frequent:custom_hsmx -> frequent:hsmx
- moved S19 35.7 mm to (214.3, 81.9)
- moved S11 35.7 mm to (127.1, 67.2)
- moved D10 35.7 mm to (114.2, 87.5)
- moved MCU1 35.7 mm to (154.8, 109.6)
- moved S17 35.7 mm to (224.8, 59.0)
- moved S25 35.7 mm to (182.5, 102.8)
- moved S10 35.7 mm to (116.9, 83.3)
- moved D11 35.7 mm to (124.4, 71.5)
- moved S12 35.7 mm to (127.0, 102.8)
- moved D19 35.7 mm to (217.0, 86.1)
- moved D12 35.7 mm to (124.3, 107.0)
- moved D6 35.7 mm to (92.6, 86.1)
- moved S2 35.7 mm to (59.4, 63.8)
- moved D15 35.7 mm to (252.1, 68.4)
- moved S20 35.7 mm to (204.1, 65.8)
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Routing:
- net P10: track 41.5 -> 255.9 mm, vias 0 -> 3
- net P3: track 100.0 -> 273.1 mm, vias 2 -> 5
- net P1: track 99.8 -> 271.6 mm, vias 2 -> 5
- net P4: track 145.6 -> 315.9 mm, vias 3 -> 5
- net P0: track 133.6 -> 279.9 mm, vias 2 -> 5
- net P2: track 152.1 -> 282.0 mm, vias 3 -> 5
- net P5: track 151.9 -> 270.8 mm, vias 2 -> 5
- net P9: track 61.3 -> 179.8 mm, vias 0 -> 3
- net P8: track 135.3 -> 203.1 mm, vias 1 -> 4
- net P7: track 218.1 -> 198.1 mm, vias 2 -> 3
- net P6: track 202.6 -> 199.5 mm
