File: kicad/metasepia_v3.kicad_pcb (KiCad board)
At the start: 2 copper layers, 227.9 x 132.7 mm, 35 parts

Commit message: wire metasepia3, create slider footprint, update footprints
Parts:
- added D1: , frequent:ComboDiode, F.Cu at (105.1, 118.3)
- added D10: , frequent:ComboDiode, F.Cu at (162.0, 136.7)
- added D11: , frequent:ComboDiode, F.Cu at (172.4, 120.8)
- added D12: , frequent:ComboDiode, F.Cu at (172.0, 156.3)
- added D13: , frequent:ComboDiode, F.Cu at (182.3, 140.4)
- added D14: , frequent:ComboDiode, F.Cu at (314.0, 118.3)
- added D15: , frequent:ComboDiode, F.Cu at (308.4, 100.1)
- added D16: , frequent:ComboDiode, F.Cu at (297.5, 129.3)
- added D17: , frequent:ComboDiode, F.Cu at (289.5, 112.1)
- added D18: , frequent:ComboDiode, F.Cu at (281.5, 94.8)
- added D19: , frequent:ComboDiode, F.Cu at (278.4, 134.2)
- added D2: , frequent:ComboDiode, F.Cu at (110.6, 100.1)
- added D20: , frequent:ComboDiode, F.Cu at (268.9, 117.8)
- added D21: , frequent:ComboDiode, F.Cu at (259.4, 101.3)
- added D22: , frequent:ComboDiode, F.Cu at (267.4, 152.7)
- added D23: , frequent:ComboDiode, F.Cu at (257.0, 136.7)
- added D24: , frequent:ComboDiode, F.Cu at (246.7, 120.8)
- added D25: , frequent:ComboDiode, F.Cu at (247.1, 156.3)
- added D26: , frequent:ComboDiode, F.Cu at (236.7, 140.4)
- added D27: , frequent:ComboDiode, F.Cu at (150.5, 185.7)
- added D28: , frequent:ComboDiode, F.Cu at (160.5, 203.2)
- added D29: , frequent:ComboDiode, F.Cu at (268.6, 185.7)
- added D3: , frequent:ComboDiode, F.Cu at (121.5, 129.3)
- added D30: , frequent:ComboDiode, F.Cu at (258.6, 203.2)
- added D4: , frequent:ComboDiode, F.Cu at (129.6, 112.1)
- added D5: , frequent:ComboDiode, F.Cu at (137.6, 94.8)
- added D6: , frequent:ComboDiode, F.Cu at (140.6, 134.2)
- added D7: , frequent:ComboDiode, F.Cu at (150.1, 117.8)
- added D8: , frequent:ComboDiode, F.Cu at (159.6, 101.3)
- added D9: , frequent:ComboDiode, F.Cu at (151.7, 152.7)
- added REF**: slider, frequent:slider, F.Cu at (209.8, 139.1)
- _1, _2, _3, _4: footprint frequent:m2hole -> m2hole
- moved S26 10.4 mm to (234.6, 137.0)
- moved S7 10.4 mm to (152.1, 114.3)
- moved S27 10.4 mm to (153.5, 183.0)
- moved _1 10.4 mm to (124.2, 96.3)
- moved S15 10.4 mm to (307.2, 96.3)
- moved S20 10.4 mm to (266.9, 114.3)
- moved S25 10.4 mm to (244.9, 153.0)
- moved S17 10.4 mm to (287.8, 108.4)
- moved S30 10.4 mm to (254.9, 201.6)
- moved S12 10.4 mm to (174.1, 153.0)
- moved S28 10.4 mm to (164.2, 201.6)
- moved S24 10.4 mm to (244.5, 117.4)
- moved S21 10.4 mm to (257.4, 97.8)
- moved S14 10.4 mm to (312.8, 114.5)
- moved _2 10.4 mm to (294.9, 96.3)
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Routing:
- net P5: track 0.00 -> 335.8 mm, vias 0 -> 4
- net P4: track 0.00 -> 316.5 mm, vias 0 -> 3
- net P2: track 0.00 -> 267.7 mm, vias 0 -> 5
- net P3: track 0.00 -> 265.1 mm, vias 0 -> 5
- net P10: track 0.00 -> 248.8 mm, vias 0 -> 2
- net P0: track 0.00 -> 240.2 mm, vias 0 -> 4
- net P1: track 0.00 -> 236.7 mm, vias 0 -> 5
- net P8: track 0.00 -> 235.8 mm, vias 0 -> 3
- net P6: track 0.00 -> 177.0 mm, vias 0 -> 3
- net P7: track 0.00 -> 174.0 mm, vias 0 -> 2
- net P9: track 0.00 -> 165.3 mm, vias 0 -> 3
- net pinky_home: track 0.00 -> 10.9 mm
- net mirror_tucky_default: track 0.00 -> 9.83 mm
- net pinky_top: track 0.00 -> 9.61 mm
- net reachy_default: track 0.00 -> 9.59 mm
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- added copper zone on B.Cu, net GND
- added copper zone on F.Cu, net GND
Other:
- outline, holes or cut-outs redrawn
