File: kicad/v4/metasepia_v4.kicad_pcb (KiCad board)
At the start: 2 copper layers, 238.7 x 131.2 mm, 70 parts

Commit message: metasepia5 create
Parts:
- removed T1: , E73:SPDT_C128955
- removed _1, _2, _3, _4: , m2hole
- added D33: , frequent:slider, F.Cu at (212.2, 135.7)
- added S33: , frequent:bat, F.Cu at (180.0, 166.4)
- added S34: , frequent:bat, F.Cu at (244.5, 166.4)
- D1, D10, D11, D12, D13, D14, D15, D16, D17, D18, D19, D2, D20, D21, D22, D23, D24, D25, D26, D27, D28, D29, D3, D30, D31, D32, D4, D5, D6, D7, D8, D9: footprint ComboDiode -> frequent:ComboDiode
- S1, S10, S11, S12, S13, S14, S15, S16, S17, S18, S19, S2, S20, S21, S22, S23, S24, S25, S26, S27, S28, S29, S3, S30, S31, S32, S4, S5, S6, S7, S8, S9: footprint MX -> frequent:MX
- moved S23 29.5 mm to (263.6, 88.7), turned to 26 degrees
- moved D23 29.2 mm to (265.4, 92.3), turned to 26 degrees
- moved S20 29.0 mm to (284.7, 83.6), turned to 23 degrees
- moved D20 28.8 mm to (286.3, 87.3), turned to 23 degrees
- moved S22 28.2 mm to (271.9, 105.8), turned to 26 degrees
- moved D22 27.9 mm to (273.7, 109.4), turned to 26 degrees
- moved S17 27.9 mm to (311.5, 87.4), turned to 16 degrees
- moved S19 27.7 mm to (292.2, 101.1), turned to 23 degrees
- moved D17 27.6 mm to (312.6, 91.3), turned to 16 degrees
- moved D19 27.4 mm to (293.7, 104.8), turned to 23 degrees
- moved S21 26.9 mm to (280.3, 122.9), turned to 26 degrees
- moved S16 26.6 mm to (316.7, 105.7), turned to 16 degrees
- moved D21 26.6 mm to (282.0, 126.5), turned to 26 degrees
- moved S18 26.4 mm to (299.6, 118.6), turned to 23 degrees
- moved D27 26.4 mm to (247.6, 143.7)
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Connections:
- MCU1 pad 17: GND -> (no net)
Other:
- board size 238.7 x 131.2 mm -> 244.8 x 308.6 mm
- net class Default removed
