File: kicad/v5/metasepia_switchplate.kicad_pcb (KiCad board)
At the start: 2 copper layers, 240.6 x 132 mm, 0 parts

Commit message: metasepia5 finish
Other:
- board size 240.6 x 132 mm -> 240.6 x 131.9 mm
- net class Default removed
