File: kicad/v5/metasepia_switchplate.kicad_pcb (KiCad board)
At the start: 2 copper layers, 240.6 x 131.9 mm, 0 parts

Commit message: work on plate and change pcb accordingly
Parts:
- added G***: LOGO, LOGO, F.Cu at (203.4, 163.5)
- added G***: LOGO, LOGO, B.Cu at (203.5, 163.3)
- added REF**: Untitled, art:METASEPIA, F.Cu at (204.4, 169.0)
Other:
- board size 240.6 x 131.9 mm -> 240.8 x 132.1 mm
