File: kicad/v5/metasepia_v5.kicad_pcb (KiCad board)
At the start: 2 copper layers, 240.6 x 131.9 mm, 68 parts

Commit message: pogo footprint part 1, begin tracing
Parts:
- MCU1: footprint frequent:xiao-smd -> frequent:xiao-pogo
- moved B1 56.6 mm to (136.8, 162.2)
- moved D26 55.7 mm to (188.8, 137.7)
- moved D23 55.7 mm to (203.4, 118.9)
- moved D20 55.7 mm to (224.3, 113.8)
- moved D1 55.7 mm to (39.5, 154.4)
- moved S9 55.7 mm to (98.9, 115.3)
- moved S29 55.7 mm to (94.8, 201.2)
- moved D17 55.7 mm to (250.6, 117.8)
- moved D27 55.7 mm to (185.7, 170.2)
- moved D30 55.7 mm to (102.8, 221.5)
- moved S7 55.7 mm to (82.3, 149.4)
- moved S4 55.7 mm to (63.0, 145.1)
- moved D14 55.7 mm to (124.4, 153.8)
- moved S14 55.7 mm to (126.4, 150.3)
- moved D19 55.7 mm to (231.8, 131.3)
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Routing:
- net P7: track 0.00 -> 153.2 mm
- net P8: track 0.00 -> 122.9 mm
- net P0: track 0.00 -> 103.6 mm, vias 0 -> 1
- net P1: track 0.00 -> 99.8 mm
- net P2: track 0.00 -> 99.5 mm
- net P5: track 0.00 -> 83.1 mm
- net P4: track 0.00 -> 81.2 mm
- net P6: track 0.00 -> 81.1 mm
- net P3: track 0.00 -> 75.4 mm
- net P10: track 0.00 -> 63.3 mm
- net P9: track 0.00 -> 61.1 mm
- net slider: track 0.00 -> 45.0 mm
- net GND: track 0.00 -> 6.20 mm
- net RST: track 0.00 -> 6.20 mm
- net BAT_POS: track 0.00 -> 6.00 mm
Other:
- board size 240.6 x 131.9 mm -> 240.6 x 132 mm

Commit message: more metasepia5 routing, fix net issue in ergogen
ergogen: must explicitly be `colrow` in pcb section
Parts:
- removed D33: , frequent:slider
- added J1: slider, frequent:slider, F.Cu at (172.2, 181.2)
- moved B1 29.7 mm to (159.7, 181.2)
- moved D26 28.9 mm to (210.7, 156.7)
- moved D27 28.9 mm to (207.5, 189.2)
- moved D30 28.9 mm to (124.6, 240.4)
- moved S10 28.9 mm to (116.6, 186.1)
- moved S6 28.9 mm to (99.7, 129.1)
- moved S17 28.9 mm to (271.4, 132.9)
- moved D23 28.9 mm to (225.3, 137.8)
- moved S26 28.9 mm to (208.7, 153.2)
- moved D19 28.9 mm to (253.6, 150.3)
- moved S18 28.9 mm to (259.5, 164.1)
- moved S9 28.9 mm to (120.8, 134.2)
- moved S24 28.9 mm to (227.7, 186.1)
- moved D11 28.9 mm to (124.1, 173.1)
- moved S3 28.9 mm to (72.9, 132.9)
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Connections:
- D1 pad 2: (no net) -> pinky_bottom
- D10 pad 2: (no net) -> index_bottom
- D11 pad 2: (no net) -> index_home
- D12 pad 2: (no net) -> index_top
- D13 pad 2: (no net) -> inner_home
- D14 pad 2: (no net) -> inner_top
- D15 pad 1: P6 -> P10
- D15 pad 2: (no net) -> mirror_pinky_bottom
- D16 pad 2: (no net) -> mirror_pinky_home
- D17 pad 2: (no net) -> mirror_pinky_top
- D18 pad 2: (no net) -> mirror_ring_bottom
- D19 pad 2: (no net) -> mirror_ring_home
- D2 pad 2: (no net) -> pinky_home
- D20 pad 2: (no net) -> mirror_ring_top
- D21 pad 2: (no net) -> mirror_middle_bottom
- D22 pad 2: (no net) -> mirror_middle_home
- D23 pad 2: (no net) -> mirror_middle_top
- D24 pad 2: (no net) -> mirror_index_bottom
- D25 pad 2: (no net) -> mirror_index_home
- D26 pad 2: (no net) -> mirror_index_top
- D27 pad 2: (no net) -> mirror_inner_home
- D28 pad 2: (no net) -> mirror_inner_top
- D29 pad 2: (no net) -> tucky_default
- D3 pad 2: (no net) -> pinky_top
- D30 pad 2: (no net) -> reachy_default
- D31 pad 2: (no net) -> mirror_tucky_default
- D32 pad 2: (no net) -> mirror_reachy_default
- D4 pad 2: (no net) -> ring_bottom
- D5 pad 2: (no net) -> ring_home
- D6 pad 2: (no net) -> ring_top
- D7 pad 2: (no net) -> middle_bottom
- D8 pad 2: (no net) -> middle_home
- MCU1 pad 18: (no net) -> RST
- S1 pad 2: (no net) -> pinky_bottom
- S10 pad 2: (no net) -> index_bottom
- S11 pad 2: (no net) -> index_home
- S12 pad 2: (no net) -> index_top
- S13 pad 2: (no net) -> inner_home
- S14 pad 2: (no net) -> inner_top
- S15 pad 1: P0 -> P1
- S15 pad 2: (no net) -> mirror_pinky_bottom
- S16 pad 2: (no net) -> mirror_pinky_home
- S17 pad 2: (no net) -> mirror_pinky_top
- S18 pad 2: (no net) -> mirror_ring_bottom
- S19 pad 2: (no net) -> mirror_ring_home
- S2 pad 2: (no net) -> pinky_home
- S20 pad 2: (no net) -> mirror_ring_top
- S21 pad 2: (no net) -> mirror_middle_bottom
- S22 pad 2: (no net) -> mirror_middle_home
- S23 pad 2: (no net) -> mirror_middle_top
- S24 pad 2: (no net) -> mirror_index_bottom
- S25 pad 2: (no net) -> mirror_index_home
- S26 pad 2: (no net) -> mirror_index_top
- S27 pad 2: (no net) -> mirror_inner_home
- S28 pad 2: (no net) -> mirror_inner_top
- S29 pad 2: (no net) -> tucky_default
- S3 pad 2: (no net) -> pinky_top
- S30 pad 2: (no net) -> reachy_default
- S31 pad 2: (no net) -> mirror_tucky_default
- S32 pad 2: (no net) -> mirror_reachy_default
- S4 pad 2: (no net) -> ring_bottom
- S5 pad 2: (no net) -> ring_home
- S6 pad 2: (no net) -> ring_top
- S7 pad 2: (no net) -> middle_bottom
- S8 pad 2: (no net) -> middle_home
- S9 pad 2: (no net) -> middle_top
Routing:
- net P6: track 81.1 -> 215.5 mm, vias 0 -> 3
- net P0: track 103.6 -> 200.7 mm, vias 1 -> 2
- net P2: track 99.5 -> 192.8 mm, vias 0 -> 3
- net P5: track 83.1 -> 139.3 mm, vias 0 -> 2
- net P4: track 81.2 -> 128.5 mm, vias 0 -> 2
- net P3: track 75.4 -> 114.5 mm, vias 0 -> 2
- net P1: track 99.8 -> 136.6 mm, vias 0 -> 2
- net P7: track 153.2 -> 187.0 mm, vias 0 -> 2
- net RST: track 6.20 -> 29.5 mm, vias 0 -> 1
- net P8: track 122.9 -> 144.5 mm, vias 0 -> 1
- net P10: track 63.3 -> 84.3 mm
- net BAT_POS: track 6.00 -> 19.9 mm, vias 0 -> 1
- net tucky_default: track 0.00 -> 9.93 mm
- net inner_top: track 0.00 -> 9.64 mm
- net inner_home: track 0.00 -> 9.63 mm
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
Commit message: xiao-pogo fp and a bit of routing
Parts:
- removed D28: , frequent:ComboDiode
- added D27: , frequent:ComboDiode, F.Cu at (190.4, 194.8)
- moved D15 60.0 mm to (267.1, 231.2), turned to -9 degrees
- moved S15 59.5 mm to (267.7, 227.2), turned to -9 degrees
- moved D16 57.9 mm to (270.1, 212.4), turned to -9 degrees
- moved S16 57.6 mm to (270.7, 208.5), turned to -9 degrees
- moved D17 56.9 mm to (273.1, 193.7), turned to -9 degrees
- moved S17 56.8 mm to (273.7, 189.7), turned to -9 degrees
- moved D18 50.5 mm to (249.6, 216.9), turned to -2 degrees
- moved S18 49.8 mm to (249.7, 212.9), turned to -2 degrees
- moved D19 47.8 mm to (250.2, 197.9), turned to -2 degrees
- moved S19 47.3 mm to (250.4, 193.9), turned to -2 degrees
- moved D20 46.4 mm to (250.9, 178.9), turned to -2 degrees
- moved S20 46.3 mm to (251.0, 174.9), turned to -2 degrees
- moved D32 45.7 mm to (181.4, 265.3), turned to 42 degrees
- moved D31 44.5 mm to (198.6, 254.0), turned to 22 degrees
- moved S32 44.0 mm to (178.7, 262.3), turned to 42 degrees
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Routing:
- net P4: track 128.5 -> 213.2 mm
- net P1: track 136.6 -> 217.9 mm, vias 2 -> 3
- net P0: track 200.7 -> 276.4 mm, vias 2 -> 3
- net P8: track 144.5 -> 181.1 mm, vias 1 -> 2
- net P10: track 84.3 -> 118.0 mm
- net P3: track 114.5 -> 141.4 mm
- net P9: track 69.3 -> 81.3 mm
- net P5: track 139.3 -> 148.3 mm
- net P2: track 192.8 -> 191.1 mm
- net slider: track 43.2 -> 44.0 mm, vias 1 -> 2
- net BAT_POS: track 19.9 -> 20.8 mm, vias 1 -> 2
Other:
- board size 240.6 x 132 mm -> 226.6 x 180.1 mm

Commit message: almost finish routing v5
Parts:
- removed D9: , frequent:ComboDiode
- added D8: , frequent:ComboDiode, F.Cu at (170.0, 92.6)
- moved D15 122.9 mm to (333.9, 128.1), turned to 16 degrees
- moved S15 121.9 mm to (332.8, 124.2), turned to 16 degrees
- moved D16 118.2 mm to (328.7, 109.8), turned to 16 degrees
- moved S16 117.2 mm to (327.6, 106.0), turned to 16 degrees
- moved D17 113.9 mm to (323.5, 91.6), turned to 16 degrees
- moved D32 113.5 mm to (270.6, 195.2), turned to 67 degrees
- moved D18 113.2 mm to (312.0, 122.5), turned to 23 degrees
- moved S17 113.0 mm to (322.4, 87.7), turned to 16 degrees
- moved D31 112.6 mm to (281.5, 177.7), turned to 47 degrees
- moved S18 112.0 mm to (310.4, 118.9), turned to 23 degrees
- moved S32 111.8 mm to (267.0, 193.6), turned to 67 degrees
- moved S31 110.9 mm to (278.6, 174.9), turned to 47 degrees
- moved D19 107.6 mm to (304.6, 105.1), turned to 23 degrees
- moved S19 106.5 mm to (303.0, 101.4), turned to 23 degrees
- moved D21 106.2 mm to (292.9, 126.7), turned to 26 degrees
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Connections:
- D27 pad 2: mirror_inner_home -> mirror_inner_top
Routing:
- net P5: track 148.3 -> 307.8 mm, vias 2 -> 5
- net P10: track 118.0 -> 263.8 mm, vias 0 -> 3
- net P4: track 213.2 -> 324.9 mm, vias 2 -> 4
- net P3: track 141.4 -> 252.0 mm, vias 2 -> 5
- net P9: track 81.3 -> 172.9 mm, vias 0 -> 3
- net P2: track 191.1 -> 261.9 mm, vias 3 -> 5
- net P1: track 217.9 -> 277.3 mm, vias 3 -> 5
- net P8: track 181.1 -> 233.0 mm, vias 2 -> 4
- net P0: track 276.4 -> 283.1 mm, vias 3 -> 5
- net P7: track 187.0 -> 188.0 mm
- added copper zone on B.Cu, net GND
- added copper zone on F.Cu, net GND
Other:
- board size 226.6 x 180.1 mm -> 240.6 x 131.9 mm

Commit message: metasepia5 finish
Parts:
- added G***: LOGO, LOGO, F.Cu at (192.7, 157.2)
- added G***: LOGO, LOGO, F.Cu at (325.1, 113.8)
- added G***: LOGO, LOGO, B.Cu at (279.2, 113.8)
- added G***: LOGO, LOGO, B.Cu at (163.2, 109.8)
- added REF**: Untitled, art:METASEPIA, F.Cu at (223.6, 159.3)
- added REF**: tism, art:tism, F.Cu at (223.5, 124.6)
- moved D20 1.12 mm to (297.6, 86.5)
- moved D23 1.12 mm to (276.7, 91.6)
- moved D27 1.12 mm to (258.9, 142.9)
- moved D31 1.12 mm to (281.9, 176.6)
- moved S23 1.12 mm to (274.9, 88.0)
- moved D13 1.12 mm to (188.2, 142.9)
- moved J1 1.12 mm to (223.5, 134.9)
- moved S10 1.12 mm to (168.0, 139.8)
- moved S11 1.12 mm to (177.5, 123.4)
- moved S13 1.12 mm to (190.2, 139.5)
- moved S14 1.12 mm to (199.7, 123.0)
- moved S29 1.12 mm to (168.1, 173.9)
- moved S8 1.12 mm to (163.8, 105.0)
- moved B1 1.12 mm to (211.1, 134.9)
- moved D29 1.12 mm to (165.2, 176.6)
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Routing:
- net GND: track 6.20 -> 66.9 mm, vias 0 -> 54
- net (no net): track 0.00 -> 6.00 mm
