File: kicad/v5/metasepia_v5.kicad_pcb (KiCad board)
At the start: 2 copper layers, 240.6 x 131.9 mm, 73 parts, among them J1 slider

Commit message: tweak pcb grounding
Routing:
- net RST: track 40.1 -> 38.6 mm
- net GND: vias 53 -> 24
