File: v7/metasepia_switchplate.kicad_pcb (KiCad board)
At the start: 2 copper layers, 237.4 x 120.8 mm, 0 parts

Commit message: finish v7 and switchplate, create production files
Parts:
- added G***: LOGO, LOGO, F.Cu at (167.1, 128.6)
- added G***: LOGO, LOGO, F.Cu at (168.7, 126.1)
- added G***: LOGO, LOGO, B.Cu at (167.2, 128.4)
- added G***: LOGO, LOGO, B.Cu at (165.9, 126.6)
- added REF**: Untitled, art:METASEPIA, F.Cu at (167.1, 108.4)
- added REF**: Untitled, art:METASEPIA, B.Cu at (167.1, 108.4)
