File: v7/metasepia_v7.kicad_pcb (KiCad board)
At the start: 2 copper layers, 237.4 x 120.8 mm, 66 parts

Commit message: Add artwork and update footprints on PCB
Added 'METASEPIA', 'LOGO', and 'tism' artwork footprints to the PCB. Adjusted the position of the SW_TACT_ALPS_SKQGABE010 footprint. Deleted the metasepia_switchplate.kicad_pro project file and updated metasepia_v7.kicad_pro project settings.
Parts:
- added G***: LOGO, LOGO, F.Cu at (314.2, 104.0)
- added G***: LOGO, LOGO, F.Cu at (193.1, 201.7)
- added G***: LOGO, LOGO, B.Cu at (162.6, 46.5)
- added REF**: Untitled, art:METASEPIA, F.Cu at (219.5, 172.5)
- added REF**: tism, art:tism, F.Cu at (219.5, 129.3)
- moved S24 0.26 mm to (274.2, 150.9)
- moved S12 0.26 mm to (183.9, 118.0)
- moved D21 0.26 mm to (288.1, 137.1)
- moved S11 0.26 mm to (174.4, 134.4)
- moved S14 0.26 mm to (197.1, 133.2)
- moved D8 0.26 mm to (160.5, 120.6)
- moved D10 0.26 mm to (162.7, 154.8)
- moved MCU1 0.26 mm to (219.6, 123.7)
- moved D20 0.26 mm to (289.9, 98.2)
- moved D32 0.26 mm to (276.8, 196.7)
- moved D23 0.26 mm to (269.1, 104.2)
- moved S10 0.26 mm to (164.9, 150.9)
- moved S4 0.26 mm to (134.0, 128.1)
- moved D13 0.26 mm to (185.3, 153.6)
- moved D29 0.26 mm to (151.1, 180.5)
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Routing:
- net P1: track 267.7 -> 273.6 mm
- net P0: track 291.9 -> 286.4 mm
- net P5: track 313.8 -> 312.0 mm
- net P3: track 262.5 -> 260.8 mm
- net P2: track 255.6 -> 254.4 mm
- net P4: vias 6 -> 5
- net GND: vias 35 -> 34
Other:
- board text added: "BOO"

Commit message: finish v7 and switchplate, create production files
Parts:
- removed the G*** at (193.1, 201.7)
- removed the G*** at (162.6, 46.5)
- added BT1: Battery_Cell, trochilidae:BatteryPadsReversible, F.Cu at (216.3, 137.1)
- added G***: LOGO, LOGO, F.Cu at (248.0, 166.4)
- added G***: LOGO, LOGO, F.Cu at (189.8, 168.0)
- added G***: LOGO, LOGO, B.Cu at (201.7, 117.6)
- added G***: LOGO, LOGO, B.Cu at (228.8, 158.5)
- moved B1 2.55 mm to (220.6, 125.2), turned to 90 degrees
- moved REF** 2.40 mm to (219.5, 131.7)
- moved G*** 1.92 mm to (314.5, 102.1)
Routing:
- net BAT_POS: track 0.00 -> 13.1 mm, vias 0 -> 2
- net RST: track 9.47 -> 10.8 mm
- net (no net): vias 0 -> 2
Other:
- board text added: "CINEMA"
- board text added: "PLUH"
- board text added: "meow"
